File: cerkit16.kicad_pcb (KiCad board)
At the start: 2 copper layers, 33 parts, among them U1 ProMicro

Commit message: updated PCB
Parts:
- added RST1: TestPoint_Small, TestPoint:TestPoint_Pad_1.5x1.5mm, B.Cu at (75.4, 70.6)
- added RST2: TestPoint_Small, TestPoint:TestPoint_Pad_1.5x1.5mm, B.Cu at (79.4, 70.6)
Connections:
- U1 pad 3: Net-(U1-Pad3) -> GND
- U1 pad 4: Net-(U1-Pad4) -> GND
Routing:
- net RST: track 0.00 -> 3.31 mm
- net GND: vias 1 -> 0
Other:
- board text added: "cerkit16 v1"
- board text added: "github.com/cerkit/kbd_cerkit16"

Commit message: cleaned up PCB
Parts:
- moved U1 0.48 mm to (88.6, 60.3)
Routing:
- net COL0: track 107.2 -> 110.1 mm, vias 1 -> 2
- net COL1: track 91.2 -> 92.4 mm, vias 1 -> 2
